File: 8266prog.sch (KiCad schematic (older format))
At the start: 4 parts, among them J1 ESP-M2, J2 USB_Ser, SW1 Reset, SW2 Program

Commit message: was a Balls up, re-do
Connections:
- net at J1.1 (Pin_1): now also J2.1 (Pin_1), SW1.2, SW2.1 (A); no longer J2.4 (Pin_4)
- net at J1.2 (Pin_2): now also J2.4 (Pin_4); no longer SW1.1
- net at J1.3 (Pin_3): now also J2.5 (Pin_5); no longer SW2.1 (A)
- net at J1.4 (Pin_4): now also SW2.2 (B); no longer J2.2 (Pin_2)
- net at J1.5 (Pin_5): now also SW1.1; no longer J2.3 (Pin_3)
- new net: J1.6 (Pin_6), J2.3 (Pin_3)
- now unconnected: J2.6 (Pin_6)
Changed lines of the file:
@@
 L conn:Conn_01x06_Female J1
 U 1 1 609ABD6A
-P 2400 2850
-F 0 "J1" H 2292 3235 50  0000 C CNN
-F 1 "ESP-M2" H 2292 3144 50  0000 C CNN
-F 2 "Connector_PinSocket_2.54mm:PinSocket_1x06_P2.54mm_Horizontal" H 2400 2850 50  0001 C CNN
-F 3 "~" H 2400 2850 50  0001 C CNN
-	1    2400 2850
-	-1   0    0    -1
+P 2400 2950
+F 0 "J1" H 2292 3335 50  0000 C CNN
+F 1 "ESP-M2" H 2292 3244 50  0000 C CNN
+F 2 "Connector_PinSocket_2.54mm:PinSocket_1x06_P2.54mm_Horizontal" H 2400 2950 50  0001 C CNN
+F 3 "~" H 2400 2950 50  0001 C CNN
+	1    2400 2950
+	-1   0    0    1
 $EndComp
 $Comp
 L conn:Conn_01x06_Female J2
 U 1 1 609AE72F
-P 4450 2850
-F 0 "J2" H 4250 3250 50  0000 L CNN
-F 1 "USB_Ser" H 4150 3150 50  0000 L CNN
-F 2 "Connector_PinSocket_2.54mm:PinSocket_1x06_P2.54mm_Horizontal" H 4450 2850 50  0001 C CNN
-F 3 "~" H 4450 2850 50  0001 C CNN
-	1    4450 2850
-	1    0    0    -1
+P 4450 2950
+F 0 "J2" H 4250 3350 50  0000 L CNN
+F 1 "USB_Ser" H 4150 3250 50  0000 L CNN
+F 2 "Connector_PinSocket_2.54mm:PinSocket_1x06_P2.54mm_Horizontal" H 4450 2950 50  0001 C CNN
+F 3 "~" H 4450 2950 50  0001 C CNN
+	1    4450 2950
+	1    0    0    1
 $EndComp
 $Comp
@@
 U 1 1 609B0195
 P 3200 2850
-F 0 "SW2" H 3550 2900 50  0000 C CNN
-F 1 "Program" H 3600 2850 50  0000 C CNN
+F 0 "SW2" H 2850 2900 50  0000 C CNN
+F 1 "Program" H 2800 2850 50  0000 C CNN
 F 2 "TrevM:SlideSwitch" H 3200 2850 50  0001 C CNN
 F 3 "~" H 3200 2850 50  0001 C CNN
 	1    3200 2850
-	1    0    0    -1
+	-1   0    0    -1
 $EndComp
 Wire Wire Line
