File: 8266prog.kicad_pcb (KiCad board)
At the start: 2 copper layers, 40.3 x 16.5 mm, 4 parts, among them J1 ESP-M2, J2 USB_Ser, SW1 Reset, SW2 Program

Commit message: was a Balls up, re-do
Parts:
- moved J2 22.7 mm to (114.3, 88.9), turned to 0 degrees
- moved J1 22.6 mm to (133.0, 101.6), turned to 180 degrees
Connections:
- J2 pad 1: (no net) -> Net-(J1-Pad1)
- J2 pad 2: Net-(J1-Pad4) -> (no net)
- J2 pad 3: Net-(J1-Pad5) -> Net-(J1-Pad6)
- J2 pad 4: Net-(J1-Pad1) -> Net-(J1-Pad2)
- J2 pad 5: (no net) -> Net-(J1-Pad3)
- J2 pad 6: Net-(J1-Pad6) -> (no net)
- SW1 pad 1: Net-(J1-Pad2) -> Net-(J1-Pad5)
- SW1 pad 2: Net-(J1-Pad6) -> Net-(J1-Pad1)
- SW2 pad 1: Net-(J1-Pad3) -> Net-(J1-Pad1)
- SW2 pad 2: Net-(J1-Pad6) -> Net-(J1-Pad4)
Routing:
- net Net-(J1-Pad6): track 44.8 -> 22.0 mm
- net Net-(J1-Pad1): track 21.1 -> 40.7 mm
- net Net-(J1-Pad2): track 16.1 -> 28.5 mm
- net Net-(J1-Pad3): track 15.8 -> 20.9 mm
- net Net-(J1-Pad5): track 19.8 -> 16.1 mm
- net Net-(J1-Pad4): track 25.2 -> 23.4 mm
Other:
- board size 40.3 x 16.5 mm -> 29 x 16.5 mm
- board text added: "3V3"
- board text added: "CTS"
- board text added: "DTR"
- board text added: "FLASH"
- board text added: "GND"
- board text added: "RESET"
- board text added: "RX"
- board text added: "TX"
- board text added: "VCC"
- board text removed: "ESP"
- board text removed: "USB"

Commit message: Minor tweaks, then created, works ok
Routing:
- net Net-(J1-Pad5): track 16.1 -> 17.4 mm
- net Net-(J1-Pad1): track 40.7 -> 40.1 mm
Other:
- board text added: "ESP"
- board text added: "USB"
